Commit message: fix turn error

File: src/description/faruk.urdf (robot description, URDF)
Before this commit: robot sam_bot, 7 links, 6 joints
Links:
- added link back_caster; collision sphere radius=${(wheel_radius+wheel_zoff-(base_height/2))}; visual sphere radius=${(wheel_radius+wheel_zoff-(base_height/2))}
Joints:
- removed joint caster_joint
- added joint back_caster_joint: type fixed, parent base_link, child back_caster, origin xyz=${-caster_xoff} 0.0 ${-(base_height/2)} rpy=0 0 0
- added joint front_caster_joint: type fixed, parent base_link, child front_caster, origin xyz=${caster_xoff} 0.0 ${-(base_height/2)} rpy=0 0 0
